File: pcb/esp32-fx.kicad_pcb (KiCad board)
At the start: 4 copper layers, 66 x 130 mm, 97 parts, among them J1 AudioJack2 (out), J2 AudioJack2 (in), J3 Jack-DC, J4 Raspberry_Pi_4, J5 AudioJack2 (in), J6 AudioJack2 (out), K1 G6K-2, Q1 MMBT2222A, Q2 MMBT2222A, Q3 MMBT2222A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

Commit message: wrote I2C I2S and using multible cores
Connections:
- C30 pad 1: /VLC -> +3.3V
- R16 pad 1: Net-(U4-AD0/~{CS}/I2S/~{LJ}) -> +3.3V
- R16 pad 2: GND -> Net-(U4-AD0/~{CS}/I2S/~{LJ})
- R21 pad 1: /VLC -> +3.3V
- R22 pad 1: /VLC -> +3.3V
- U4 pad 12: Net-(U4-AD1/CDIN/MDIV1) -> /SDIN
- U4 pad 8: /VLC -> +3.3V
