File: full-pcb/Input.kicad_sch (KiCad schematic)
At the start: 13 parts, among them U2 OPA1664D

Commit message: trouble with defmt
Parts:
- removed C13, C2: 1nf, Capacitor_SMD:C_0805_2012Metric, symbol Device:C
- removed R13, R14, R3, R4: 100, Resistor_SMD:R_0603_1608Metric, symbol Device:R
Connections:
- net AUDIO_IN_JACK_LEFT: now also C7.1, R10.2
- net AUDIO_IN_JACK_LEFT_BUF: now also U2.1, U2.2 (-)
- net AUDIO_IN_JACK_RIGHT: now also C11.1, R8.2
- net AUDIO_IN_JACK_RIGHT_BUF: now also U2.6 (-), U2.7
