File: full-pcb/Input.kicad_sch (KiCad schematic)
At the start: 7 parts, among them U2 OPA1664D

Commit message: got the fft to work YAY!
Connections:
- net AUDIO_IN_JACK_LEFT_BUF: now also U2.8, U2.9 (-); no longer U2.1, U2.2 (-)
- net at C7.2, R1.1: now also U2.10 (+); no longer U2.3 (+)
Changed lines of the file:
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@@
 		(lib_id "Amplifier_Operational:OPA1664D")
 		(at 162.56 125.73 0)
-		(unit 1)
+		(unit 3)
 		(body_style 1)
 		(exclude_from_sim no)
@@
 				(path "/ac8ee366-0662-41f8-9745-078ec3fbb21b/0ca96f51-23c0-4c17-837f-32f367c7277c"
 					(reference "U2")
-					(unit 1)
+					(unit 3)
 				)
 			)

Commit message: pedal works but is buggy
Parts:
- renumbered C11 to C3, C7 to C4, R5 to R3, R8 to R4, R1 to R5, R10 to R6, U2 to U1
Connections:
- net AUDIO_IN_JACK_LEFT_BUF: now also U1.6 (-), U1.7; no longer U1.8, U1.9 (-)
- net AUDIO_IN_JACK_RIGHT_BUF: now also U1.8, U1.9 (-); no longer U1.6 (-), U1.7
- net at C4.2, R5.1: now also U1.5 (+); no longer U1.10 (+)
- net at C3.2, R3.1: now also U1.10 (+); no longer U1.5 (+)
Changed lines of the file:
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@@
 	)
 	(global_label "AUDIO_IN_JACK_LEFT_BUF"
-		(shape input)
+		(shape output)
 		(at 182.88 125.73 0)
 		(fields_autoplaced yes)
@@
 	)
 	(global_label "AUDIO_IN_JACK_RIGHT_BUF"
-		(shape input)
+		(shape output)
 		(at 185.42 66.04 0)
 		(fields_autoplaced yes)
@@
 		(dnp no)
 		(fields_autoplaced yes)
-		(property "Reference" "#PWR07"
+		(property "Reference" "#PWR018"
 			(at 146.05 118.11 0)
 			(hide yes)
@@
 			(project "full_pcb"
 				(path "/ac8ee366-0662-41f8-9745-078ec3fbb21b/0ca96f51-23c0-4c17-837f-32f367c7277c"
-					(reference "#PWR07")
+					(reference "#PWR018")
 					(unit 1)
 				)
@@
 		(dnp no)
 		(fields_autoplaced yes)
-		(property "Reference" "R1"
+		(property "Reference" "R5"
 			(at 148.59 116.8399 0)
 			(show_name no)
@@
 			(project "full_pcb"
 				(path "/ac8ee366-0662-41f8-9745-078ec3fbb21b/0ca96f51-23c0-4c17-837f-32f367c7277c"
-					(reference "R1")
+					(reference "R5")
 					(unit 1)
 				)
@@
 		(dnp no)
 		(fields_autoplaced yes)
-		(property "Reference" "R10"
+		(property "Reference" "R6"
 			(at 135.89 129.5399 0)
 			(show_name no)
@@
 			(project "full_pcb"
 				(path "/ac8ee366-0662-41f8-9745-078ec3fbb21b/0ca96f51-23c0-4c17-837f-32f367c7277c"
-					(reference "R10")
+					(reference "R6")
 					(unit 1)
 				)
@@
 		(dnp no)
 		(fields_autoplaced yes)
-		(property "Reference" "C11"
+		(property "Reference" "C3"
 			(at 124.46 55.88 90)
 			(show_name no)
@@
 			(project "full_pcb"
 				(path "/ac8ee366-0662-41f8-9745-078ec3fbb21b/0ca96f51-23c0-4c17-837f-32f367c7277c"
-					(reference "C11")
+					(reference "C3")
 					(unit 1)
 				)
@@
 		(dnp no)
 		(fields_autoplaced yes)
-		(property "Reference" "#PWR0104"
+		(property "Reference" "#PWR017"
 			(at 115.57 77.47 0)
 			(hide yes)
@@
 			(project "full_pcb"
 				(path "/ac8ee366-0662-41f8-9745-078ec3fbb21b/0ca96f51-23c0-4c17-837f-32f367c7277c"
-					(reference "#PWR0104")
+					(reference "#PWR017")
 					(unit 1)
 				)
@@
 		(dnp no)
 		(fields_autoplaced yes)
-		(property "Reference" "R5"
+		(property "Reference" "R3"
 			(at 134.62 57.1499 0)
 			(show_name no)
@@
 			(project "full_pcb"
 				(path "/ac8ee366-0662-41f8-9745-078ec3fbb21b/0ca96f51-23c0-4c17-837f-32f367c7277c"
-					(reference "R5")
+					(reference "R3")
 					(unit 1)
 				)
@@
 		(lib_id "Amplifier_Operational:OPA1664D")
 		(at 162.56 125.73 0)
-		(unit 3)
+		(unit 2)
 		(body_style 1)
 		(exclude_from_sim no)
@@
 		(dnp no)
 		(fields_autoplaced yes)
-		(property "Reference" "U2"
+		(property "Reference" "U1"
 			(at 162.56 115.57 0)
 			(show_name no)
@@
 			(project "full_pcb"
 				(path "/ac8ee366-0662-41f8-9745-078ec3fbb21b/0ca96f51-23c0-4c17-837f-32f367c7277c"
-					(reference "U2")
-					(unit 3)
+					(reference "U1")
+					(unit 2)
 				)
 			)
@@
 		(dnp no)
 		(fields_autoplaced yes)
-		(property "Reference" "#PWR06"
+		(property "Reference" "#PWR016"
 			(at 132.08 58.42 0)
 			(hide yes)
@@
 			(project "full_pcb"
 				(path "/ac8ee366-0662-41f8-9745-078ec3fbb21b/0ca96f51-23c0-4c17-837f-32f367c7277c"
-					(reference "#PWR06")
+					(reference "#PWR016")
 					(unit 1)
 				)
@@
 		(dnp no)
 		(fields_autoplaced yes)
-		(property "Reference" "R8"
+		(property "Reference" "R4"
 			(at 118.11 66.0399 0)
 			(show_name no)
@@
 			(project "full_pcb"
 				(path "/ac8ee366-0662-41f8-9745-078ec3fbb21b/0ca96f51-23c0-4c17-837f-32f367c7277c"
-					(reference "R8")
+					(reference "R4")
 					(unit 1)
 				)
@@
 		(dnp no)
 		(fields_autoplaced yes)
-		(property "Reference" "#PWR0106"
+		(property "Reference" "#PWR019"
 			(at 133.35 140.97 0)
 			(hide yes)
@@
 			(project "full_pcb"
 				(path "/ac8ee366-0662-41f8-9745-078ec3fbb21b/0ca96f51-23c0-4c17-837f-32f367c7277c"
-					(reference "#PWR0106")
+					(reference "#PWR019")
 					(unit 1)
 				)
@@
 		(lib_id "Amplifier_Operational:OPA1664D")
 		(at 151.13 66.04 0)
-		(unit 2)
+		(unit 3)
 		(body_style 1)
 		(exclude_from_sim no)
@@
 		(dnp no)
 		(fields_autoplaced yes)
-		(property "Reference" "U2"
+		(property "Reference" "U1"
 			(at 151.13 55.88 0)
 			(show_name no)
@@
 			(project "full_pcb"
 				(path "/ac8ee366-0662-41f8-9745-078ec3fbb21b/0ca96f51-23c0-4c17-837f-32f367c7277c"
-					(reference "U2")
-					(unit 2)
+					(reference "U1")
+					(unit 3)
 				)
 			)
@@
 		(dnp no)
 		(fields_autoplaced yes)
-		(property "Reference" "C7"
+		(property "Reference" "C4"
 			(at 138.43 115.57 90)
 			(show_name no)
@@
 			(project "full_pcb"
 				(path "/ac8ee366-0662-41f8-9745-078ec3fbb21b/0ca96f51-23c0-4c17-837f-32f367c7277c"
-					(reference "C7")
-					(unit 1)
-				)
+					(reference "C4")
+					(unit 1)
+				)
