File: full-pcb/Output.kicad_sch (KiCad schematic)
At the start: 13 parts, among them U2 OPA1664D

Commit message: trouble with defmt
Parts:
- removed C16, C17: 1nf, Capacitor_SMD:C_0805_2012Metric, symbol Device:C
- removed R25, R26, R6: 100, Resistor_SMD:R_0603_1608Metric, symbol Device:R
- removed R9: 7.5k, Resistor_SMD:R_0603_1608Metric, symbol Device:R
- added C13, C2: 2.2nf, Capacitor_SMD:C_0805_2012Metric, symbol Device:C
- added R11, R12: 2M, Resistor_SMD:R_0603_1608Metric, symbol Device:R
- added R3: 100, Resistor_SMD:R_0603_1608Metric, symbol Device:R
- added R4: 3.3K, Resistor_SMD:R_0603_1608Metric, symbol Device:R
- R2: value 7.5k -> 100; MPN C23234 -> C22775
- R7: value 100 -> 3.3K; MPN C22775 -> C22978
Connections:
- net AUDIO_OUT_JACK_LEFT: now also C6.2, R11.2
- net AUDIO_OUT_JACK_LEFT_BUF: now also R4.1
- net AUDIO_OUT_JACK_RIGHT: now also C9.2, R12.2
- net GND: now also C13.1, C2.1, R11.1, R12.1
- net at C5.1: now also C13.2, R4.2
- net at C9.1: now also R3.2
- net at C3.1, R7.2: now also C2.2
- net at U2.13 (-), U2.14: now also R3.1
Other:
- moved on the sheet: R7
