File: full-pcb/Output.kicad_sch (KiCad schematic)
At the start: 13 parts, among them U2 OPA1664D

Commit message: got the fft to work YAY!
Connections:
- net at C3.2: now also U2.3 (+); no longer U2.12 (+)
- net at C5.2: now also U2.12 (+); no longer U2.10 (+)
- new net: R2.1, U2.13 (-), U2.14
- new net: R3.1, U2.1, U2.2 (-)
Changed lines of the file:
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@@
 		(lib_id "Amplifier_Operational:OPA1664D")
 		(at 115.57 105.41 0)
-		(unit 3)
+		(unit 4)
 		(body_style 1)
 		(exclude_from_sim no)
@@
 				(path "/ac8ee366-0662-41f8-9745-078ec3fbb21b/71b17037-91e4-4ab7-a98f-0d6408c65901"
 					(reference "U2")
-					(unit 3)
+					(unit 4)
 				)
 			)
@@
 		(lib_id "Amplifier_Operational:OPA1664D")
 		(at 134.62 67.31 0)
-		(unit 4)
+		(unit 1)
 		(body_style 1)
 		(exclude_from_sim no)
@@
 				(path "/ac8ee366-0662-41f8-9745-078ec3fbb21b/71b17037-91e4-4ab7-a98f-0d6408c65901"
 					(reference "U2")
-					(unit 4)
-				)
-			)
+					(unit 1)
+				)
+			)

Commit message: pedal works but is buggy
Parts:
- renumbered C13 to C10, C3 to C5, C9 to C6, C2 to C7, C5 to C8, C6 to C9, R4 to R10, R2 to R11, R11 to R12, R3 to R8, R12 to R9, U2 to U1
Connections:
- net at C5.2: now also U1.12 (+); no longer U1.3 (+)
- net at C8.2: now also U1.3 (+); no longer U1.12 (+)
- new net: R11.1, U1.1, U1.2 (-)
- new net: R8.1, U1.13 (-), U1.14
Changed lines of the file:
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@@
 	)
 	(global_label "AUDIO_OUT_JACK_RIGHT"
-		(shape input)
+		(shape output)
 		(at 195.58 67.31 0)
 		(fields_autoplaced yes)
@@
 	)
 	(global_label "AUDIO_OUT_JACK_LEFT"
-		(shape input)
+		(shape output)
 		(at 166.37 105.41 0)
 		(fields_autoplaced yes)
@@
 		(dnp no)
 		(fields_autoplaced yes)
-		(property "Reference" "C9"
+		(property "Reference" "C6"
 			(at 165.1 59.69 90)
 			(show_name no)
@@
 			(project "full_pcb"
 				(path "/ac8ee366-0662-41f8-9745-078ec3fbb21b/71b17037-91e4-4ab7-a98f-0d6408c65901"
-					(reference "C9")
+					(reference "C6")
 					(unit 1)
 				)
@@
 		(dnp no)
 		(fields_autoplaced yes)
-		(property "Reference" "C3"
+		(property "Reference" "C5"
 			(at 96.52 57.15 90)
 			(show_name no)
@@
 			(project "full_pcb"
 				(path "/ac8ee366-0662-41f8-9745-078ec3fbb21b/71b17037-91e4-4ab7-a98f-0d6408c65901"
-					(reference "C3")
+					(reference "C5")
 					(unit 1)
 				)
@@
 		(dnp no)
 		(fields_autoplaced yes)
-		(property "Reference" "R11"
+		(property "Reference" "R12"
 			(at 158.75 107.9499 0)
 			(show_name no)
@@
 			(project "full_pcb"
 				(path "/ac8ee366-0662-41f8-9745-078ec3fbb21b/71b17037-91e4-4ab7-a98f-0d6408c65901"
-					(reference "R11")
+					(reference "R12")
 					(unit 1)
 				)
@@
 		(dnp no)
 		(fields_autoplaced yes)
-		(property "Reference" "C5"
+		(property "Reference" "C8"
 			(at 81.28 95.25 90)
 			(show_name no)
@@
 			(project "full_pcb"
 				(path "/ac8ee366-0662-41f8-9745-078ec3fbb21b/71b17037-91e4-4ab7-a98f-0d6408c65901"
-					(reference "C5")
+					(reference "C8")
 					(unit 1)
 				)
@@
 		(lib_id "Amplifier_Operational:OPA1664D")
 		(at 115.57 105.41 0)
-		(unit 4)
+		(unit 1)
 		(body_style 1)
 		(exclude_from_sim no)
@@
 		(dnp no)
 		(fields_autoplaced yes)
-		(property "Reference" "U2"
+		(property "Reference" "U1"
 			(at 115.57 95.25 0)
 			(show_name no)
@@
 			(project "full_pcb"
 				(path "/ac8ee366-0662-41f8-9745-078ec3fbb21b/71b17037-91e4-4ab7-a98f-0d6408c65901"
-					(reference "U2")
-					(unit 4)
+					(reference "U1")
+					(unit 1)
 				)
 			)
@@
 		(dnp no)
 		(fields_autoplaced yes)
-		(property "Reference" "R12"
+		(property "Reference" "R9"
 			(at 177.8 69.8499 0)
 			(show_name no)
@@
 			(project "full_pcb"
 				(path "/ac8ee366-0662-41f8-9745-078ec3fbb21b/71b17037-91e4-4ab7-a98f-0d6408c65901"
-					(reference "R12")
+					(reference "R9")
 					(unit 1)
 				)
@@
 		(dnp no)
 		(fields_autoplaced yes)
-		(property "Reference" "#PWR0108"
+		(property "Reference" "#PWR021"
 			(at 175.26 81.28 0)
 			(hide yes)
@@
 			(project "full_pcb"
 				(path "/ac8ee366-0662-41f8-9745-078ec3fbb21b/71b17037-91e4-4ab7-a98f-0d6408c65901"
-					(reference "#PWR0108")
+					(reference "#PWR021")
 					(unit 1)
 				)
@@
 		(dnp no)
 		(fields_autoplaced yes)
-		(property "Reference" "#PWR049"
+		(property "Reference" "#PWR022"
 			(at 72.39 116.84 0)
 			(hide yes)
@@
 			(project "full_pcb"
 				(path "/ac8ee366-0662-41f8-9745-078ec3fbb21b/71b17037-91e4-4ab7-a98f-0d6408c65901"
-					(reference "#PWR049")
+					(reference "#PWR022")
 					(unit 1)
 				)
@@
 		(dnp no)
 		(fields_autoplaced yes)
-		(property "Reference" "R3"
+		(property "Reference" "R8"
 			(at 148.59 60.96 90)
 			(show_name no)
@@
 			(project "full_pcb"
 				(path "/ac8ee366-0662-41f8-9745-078ec3fbb21b/71b17037-91e4-4ab7-a98f-0d6408c65901"
-					(reference "R3")
+					(reference "R8")
 					(unit 1)
 				)
@@
 		(dnp no)
 		(fields_autoplaced yes)
-		(property "Reference" "C13"
+		(property "Reference" "C10"
 			(at 76.2 105.4099 0)
 			(show_name no)
@@
 			(project "full_pcb"
 				(path "/ac8ee366-0662-41f8-9745-078ec3fbb21b/71b17037-91e4-4ab7-a98f-0d6408c65901"
-					(reference "C13")
+					(reference "C10")
 					(unit 1)
 				)
@@
 		(dnp no)
 		(fields_autoplaced yes)
-		(property "Reference" "C6"
+		(property "Reference" "C9"
 			(at 151.13 97.79 90)
 			(show_name no)
@@
 			(project "full_pcb"
 				(path "/ac8ee366-0662-41f8-9745-078ec3fbb21b/71b17037-91e4-4ab7-a98f-0d6408c65901"
-					(reference "C6")
+					(reference "C9")
 					(unit 1)
 				)
@@
 		(dnp no)
 		(fields_autoplaced yes)
-		(property "Reference" "R2"
+		(property "Reference" "R11"
 			(at 135.89 99.06 90)
 			(show_name no)
@@
 			(project "full_pcb"
 				(path "/ac8ee366-0662-41f8-9745-078ec3fbb21b/71b17037-91e4-4ab7-a98f-0d6408c65901"
-					(reference "R2")
+					(reference "R11")
 					(unit 1)
 				)
@@
 		(dnp no)
 		(fields_autoplaced yes)
-		(property "Reference" "C2"
+		(property "Reference" "C7"
 			(at 91.44 68.5799 0)
 			(show_name no)
@@
 			(project "full_pcb"
 				(path "/ac8ee366-0662-41f8-9745-078ec3fbb21b/71b17037-91e4-4ab7-a98f-0d6408c65901"
-					(reference "C2")
+					(reference "C7")
 					(unit 1)
 				)
@@
 		(dnp no)
 		(fields_autoplaced yes)
-		(property "Reference" "#PWR0107"
+		(property "Reference" "#PWR023"
 			(at 156.21 119.38 0)
 			(hide yes)
@@
 			(project "full_pcb"
 				(path "/ac8ee366-0662-41f8-9745-078ec3fbb21b/71b17037-91e4-4ab7-a98f-0d6408c65901"
-					(reference "#PWR0107")
+					(reference "#PWR023")
 					(unit 1)
 				)
@@
 		(dnp no)
 		(fields_autoplaced yes)
-		(property "Reference" "R4"
+		(property "Reference" "R10"
 			(at 63.5 96.52 90)
 			(show_name no)
@@
 			(project "full_pcb"
 				(path "/ac8ee366-0662-41f8-9745-078ec3fbb21b/71b17037-91e4-4ab7-a98f-0d6408c65901"
-					(reference "R4")
+					(reference "R10")
 					(unit 1)
 				)
@@
 		(dnp no)
 		(fields_autoplaced yes)
-		(property "Reference" "#PWR038"
+		(property "Reference" "#PWR020"
 			(at 87.63 80.01 0)
 			(hide yes)
@@
 			(project "full_pcb"
 				(path "/ac8ee366-0662-41f8-9745-078ec3fbb21b/71b17037-91e4-4ab7-a98f-0d6408c65901"
-					(reference "#PWR038")
+					(reference "#PWR020")
 					(unit 1)
 				)
@@
 		(lib_id "Amplifier_Operational:OPA1664D")
 		(at 134.62 67.31 0)
-		(unit 1)
+		(unit 4)
 		(body_style 1)
 		(exclude_from_sim no)
@@
 		(dnp no)
 		(fields_autoplaced yes)
-		(property "Reference" "U2"
+		(property "Reference" "U1"
 			(at 134.62 57.15 0)
 			(show_name no)
@@
 			(project "full_pcb"
 				(path "/ac8ee366-0662-41f8-9745-078ec3fbb21b/71b17037-91e4-4ab7-a98f-0d6408c65901"
-					(reference "U2")
-					(unit 1)
-				)
-			)
+					(reference "U1")
+					(unit 4)
+				)
+			)
