File: full-pcb/full_pcb.kicad_pcb (KiCad board)
At the start: 4 copper layers, 58.5 x 60.5 mm, 66 parts, among them J1 Screw_Terminal_01x02, J3 Barrel_Jack_Switch, J4 AUDIO_IN_TRS, J5 AUDIO_OUT_TRS, J6 Screw_Terminal_01x02, P1 USB_C_Plug_USB2.0, U1 ESP32-C3-WROOM-02, U2 OPA1664D, U3 AMS1117-5.0, U4 CJ431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

Commit message: trouble with defmt
Parts:
- removed AUDIO_IN1, AUDIO_RAW1: TestPoint, TestPoint:TestPoint_Pad_D2.0mm
- removed BOOT1, RESET1: SW_Push, Button_Switch_SMD:SW_SPST_TL3342
- removed C19: 10uf, Capacitor_Tantalum_SMD:CP_EIA-3216-18_Kemet-A
- removed C20: 0.1uf, Capacitor_SMD:C_0805_2012Metric
- removed P1: USB_C_Plug_USB2.0, Connector_USB:USB_C_Receptacle_HRO_TYPE-C-31-M-17
- removed R13, R14, R25, R26, R6: 100, Resistor_SMD:R_0603_1608Metric
- removed R15: 5.1k, Resistor_SMD:R_0603_1608Metric
- removed R24, R28, R29, R30: 10k, Resistor_SMD:R_0603_1608Metric
- removed R9: 7.5k, Resistor_SMD:R_0603_1608Metric
- removed U5: AMS1117-3.3, Package_TO_SOT_SMD:SOT-223-3_TabPin2
- removed U6: USBLC6-2SC6, Package_TO_SOT_SMD:SOT-23-6
- added 5V2: TestPoint, TestPoint:TestPoint_Pad_D2.0mm, F.Cu at (84.3, 88.4)
- added D3: SS14, Diode_SMD:D_SMA, F.Cu at (217.0, 133.2)
- added J7: AUDIO_IN_TRS, Connector_Audio:Jack_6.35mm_Neutrik_NMJ6HCD3_Horizontal, F.Cu at (221.8, 43.2)
- added J8: AUDIO_OUT_TRS, Connector_Audio:Jack_6.35mm_Neutrik_NMJ6HCD3_Horizontal, F.Cu at (186.7, 59.5)
- added R11: 2M, Resistor_SMD:R_0603_1608Metric, F.Cu at (196.2, 39.2)
- added R12: 2M, Resistor_SMD:R_0603_1608Metric, F.Cu at (196.2, 42.8)
- added U7: XIAO-ESP32-C3-DIP, Seeed Studio XIAO Series Library:XIAO-ESP32-C3-DIP, F.Cu at (230.4, 125.5)
- 5V1, 9V1, A1, GND1, J1, J3, J4, J5, J6: moved to F.Cu
- C13, C2: value 1nf -> 2.2nf
- C14: value 10uf -> 0.1uf
- C15: footprint Capacitor_Tantalum_SMD:CP_EIA-3216-18_Kemet-A -> Capacitor_SMD:C_0805_2012Metric
- C16, C17: value 1nf -> 0.1uf
- C18: value 0.1uf -> 10uf
- D1: value 1N5817 -> SS34; footprint Diode_SMD:D_SOD-123 -> Diode_SMD:D_SMA
- R2: value 7.5k -> 100
- R27: value 330 -> 1K
- R4, R7: value 100 -> 3.3K
- U1: value ESP32-C3-WROOM-02 -> 78L05G-AB3-R; footprint RF_Module:ESP32-C3-WROOM-02 -> Package_TO_SOT_SMD:SOT-89-3
- moved C18 122.8 mm to (189.8, 125.5), turned to -90 degrees
- moved J4 122.7 mm to (221.8, 22.5), turned to 0 degrees
- moved C15 120.8 mm to (190.0, 133.5)
- moved R23 116.3 mm to (210.5, 39.2), turned to 0 degrees
- moved U4 115.3 mm to (210.8, 41.8), turned to 0 degrees
- moved C7 110.4 mm to (211.2, 34.3), turned to 0 degrees
- moved R10 109.1 mm to (210.2, 36.8), turned to 90 degrees
- moved C14 108.2 mm to (202.1, 46.5), turned to 180 degrees
- moved R8 108.2 mm to (210.2, 45.0), turned to -90 degrees
- moved R1 108.1 mm to (212.2, 36.8)
- moved R5 107.2 mm to (212.2, 45.0)
- moved C11 105.9 mm to (211.2, 47.5), turned to 0 degrees
- moved 5V1 104.0 mm to (84.3, 84.4), turned to 0 degrees
- moved J6 102.4 mm to (96.5, 86.5), turned to 0 degrees
- moved C12 99.1 mm to (205.9, 46.5), turned to 0 degrees
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Connections:
- C10 pad 1: +5V -> +5VD
- C11 pad 1: Net-(C11-Pad1) -> AUDIO_IN_JACK_RIGHT
- C12 pad 1: +5V -> +5VA
- C13 pad 2: Net-(U2B--) -> Net-(C13-Pad2)
- C14 pad 1: GND -> +5VA
- C14 pad 2: +5V -> GND
- C15 pad 1: +9V -> GND
- C15 pad 2: GND -> +5VA
- C16 pad 1: GND -> +5VD
- C16 pad 2: Net-(C16-Pad2) -> GND
- C17 pad 1: GND -> +5VD
- C17 pad 2: Net-(C17-Pad2) -> GND
- C18 pad 1: +9V -> GND
- C18 pad 2: GND -> +9V
- C2 pad 2: Net-(U2A--) -> Net-(C2-Pad2)
- C3 pad 1: Net-(C3-Pad1) -> Net-(C2-Pad2)
- C4 pad 1: +5V -> +5VD
- C5 pad 1: Net-(C5-Pad1) -> Net-(C13-Pad2)
- C6 pad 1: Net-(C16-Pad2) -> Net-(C6-Pad1)
- C6 pad 2: Net-(C6-Pad2) -> AUDIO_OUT_JACK_LEFT
- C7 pad 1: Net-(C7-Pad1) -> AUDIO_IN_JACK_LEFT
- C9 pad 1: Net-(C17-Pad2) -> Net-(C9-Pad1)
- C9 pad 2: Net-(C9-Pad2) -> AUDIO_OUT_JACK_RIGHT
- J4 pad R: AUDIO_IN_JACK_RIGHT -> unconnected-(J4-PadR)
- J5 pad R: AUDIO_OUT_JACK_RIGHT -> unconnected-(J5-PadR)
- R10 pad 2: Net-(C7-Pad1) -> AUDIO_IN_JACK_LEFT
- R2 pad 2: Net-(C16-Pad2) -> Net-(C6-Pad1)
- R23 pad 2: +5V -> +5VA
- R3 pad 1: Net-(C7-Pad1) -> Net-(U2D--)
- R3 pad 2: AUDIO_IN_JACK_LEFT -> Net-(C9-Pad1)
- R4 pad 1: Net-(C11-Pad1) -> AUDIO_OUT_JACK_LEFT_BUF
- R4 pad 2: AUDIO_IN_JACK_RIGHT -> Net-(C13-Pad2)
- R7 pad 2: Net-(C3-Pad1) -> Net-(C2-Pad2)
- R8 pad 2: Net-(C11-Pad1) -> AUDIO_IN_JACK_RIGHT
- U1 pad 1: +3.3V -> GND
- U1 pad 2: Net-(U1-EN) -> +5VA
- U1 pad 3: unconnected-(U1-IO4-Pad3) -> +9V
- U2 pad 1: Net-(U2A--) -> AUDIO_IN_JACK_LEFT_BUF
- U2 pad 2: Net-(U2A--) -> AUDIO_IN_JACK_LEFT_BUF
- U2 pad 4: +5V -> +5VA
- U2 pad 6: Net-(U2B--) -> AUDIO_IN_JACK_RIGHT_BUF
- U2 pad 7: Net-(U2B--) -> AUDIO_IN_JACK_RIGHT_BUF
- U3 pad 2: +5V -> +5VD
Routing:
- net +9V: track 64.2 -> 8.18 mm, vias 1 -> 0
- net +5VD: track 0.00 -> 38.1 mm
- net Net-(A1-I2C1_SCL): track 37.9 -> 0.00 mm
- net Net-(A1-I2C1_SDA): track 36.4 -> 0.00 mm, vias 2 -> 0
- net +3.3VD: track 31.8 -> 0.00 mm
- net AUDIO_IN_JACK_LEFT_BUF: track 29.7 -> 0.00 mm, vias 1 -> 0
- net GND: track 22.9 -> 0.00 mm, vias 30 -> 0
- net +2.5V: track 21.4 -> 0.00 mm, vias 3 -> 0
- net AUDIO_IN_JACK_RIGHT_BUF: track 19.6 -> 0.00 mm, vias 1 -> 0
- net +5V: track 19.6 -> 0.00 mm, vias 10 -> 0
- net AUDIO_OUT_JACK_RIGHT_BUF: track 16.8 -> 0.00 mm
- net Net-(A1-ADC_6): track 16.4 -> 0.00 mm
- net AUDIO_OUT_JACK_LEFT_BUF: track 15.6 -> 0.00 mm
- net AUDIO_IN_JACK_RIGHT: track 14.4 -> 0.00 mm
- net AUDIO_OUT_JACK_RIGHT: track 13.0 -> 0.00 mm
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- removed copper zone on F.Cu, net +5V
- removed copper zone on In2.Cu, net +5V
- removed copper zone on F.Cu, net GND
- removed copper zone on In1.Cu, net GND
- removed copper zone on F.Cu, net POWER_JACK_PWR
Other:
- board size 58.5 x 60.5 mm -> 73 x 129 mm
- board text removed: "Install 2 2.54mm 1x20 female pin headers for A1"
- board text removed: "SCL"
- board text removed: "SDA"
