File: full-pcb/full_pcb.kicad_pcb (KiCad board)
At the start: 4 copper layers, 73 x 129 mm, 53 parts, among them J1 Screw_Terminal_01x02, J3 Barrel_Jack_Switch, J4 AUDIO_IN_TRS, J5 AUDIO_OUT_TRS, J6 Screw_Terminal_01x02, J7 AUDIO_IN_TRS, J8 AUDIO_OUT_TRS, U1 78L05G-AB3-R, U2 OPA1664D, U3 AMS1117-5.0, U4 CJ431, U7 XIAO-ESP32-C3-DIP

Commit message: got the fft to work YAY!
Parts:
- removed 5V1, 5V2, 9V1, GND1, GND2: TestPoint, TestPoint:TestPoint_Pad_D2.0mm
- removed C10, C8: 0.1uf, Capacitor_SMD:C_0805_2012Metric
- removed C4: 10uf, Capacitor_Tantalum_SMD:CP_EIA-3216-18_Kemet-A
- removed D1: SS34, Diode_SMD:D_SMA
- removed U7: XIAO-ESP32-C3-DIP, Seeed Studio XIAO Series Library:XIAO-ESP32-C3-DIP
- added C19: 10uf, Capacitor_SMD:C_0805_2012Metric, F.Cu at (153.4, 153.4)
- added C20: 0.01uf, Capacitor_SMD:C_0805_2012Metric, F.Cu at (161.2, 158.0)
- added D5: SS34, Diode_SMD:D_SMA, F.Cu at (150.6, 156.8)
- added D6: SS34, Diode_SMD:D_SMA, F.Cu at (156.4, 157.9)
- added L1: 18uH, Inductor_SMD:L_6.3x6.3_H3, F.Cu at (165.7, 154.4)
- added R6: 3.24k, Resistor_SMD:R_0603_1608Metric, F.Cu at (160.3, 149.8)
- added R9: 10k, Resistor_SMD:R_0603_1608Metric, F.Cu at (163.6, 149.8)
- added U5: XIAO-ESP32-C6-DIP, Seeed Studio XIAO Series Library:XIAO-ESP32-C6-DIP, F.Cu at (182.5, 148.5)
- C1: value 10uf -> 220uf; footprint Capacitor_Tantalum_SMD:CP_EIA-3216-18_Kemet-A -> Capacitor_Tantalum_SMD:CP_EIA-7343-31_Kemet-D
- U3: value AMS1117-5.0 -> TPS5430DDA; footprint Package_TO_SOT_SMD:SOT-223-3_TabPin2 -> Package_SO:TI_SO-PowerPAD-8_ThermalVias
- moved C16 102.5 mm to (178.9, 154.8), turned to 90 degrees
- moved J6 100.8 mm to (187.8, 129.3), turned to 90 degrees
- moved C17 99.0 mm to (176.9, 154.8), turned to 90 degrees
- moved A1 87.8 mm to (137.5, 157.3), turned to 180 degrees
- moved R27 75.4 mm to (161.0, 142.1), turned to 90 degrees
- moved D2 75.2 mm to (162.8, 142.2), turned to -90 degrees
- moved R5 55.3 mm to (162.0, 68.0)
- moved R1 55.2 mm to (162.0, 59.8)
- moved C11 53.5 mm to (163.0, 70.5), turned to 180 degrees
- moved C12 53.5 mm to (157.7, 69.5)
- moved C14 53.5 mm to (153.8, 69.5)
- moved C6 53.5 mm to (149.0, 59.8)
- moved C7 53.5 mm to (163.0, 57.3), turned to 180 degrees
- moved C9 53.5 mm to (149.0, 68.2)
- moved J4 53.5 mm to (173.5, 45.5)
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Connections:
- A1 pad 10: unconnected-(A1-SPI1_POCI-Pad10) -> POCI
- A1 pad 11: unconnected-(A1-SPI1_PICO-Pad11) -> PICO
- A1 pad 14: DAISY_OUT -> unconnected-(A1-USART1_TX-Pad14)
- A1 pad 15: DAISY_IN -> unconnected-(A1-USART1_RX-Pad15)
- A1 pad 38: unconnected-(A1-3V3_D-Pad38) -> +3.3VD
- A1 pad 8: unconnected-(A1-SPI1_CS-Pad8) -> GND
- A1 pad 9: unconnected-(A1-SPI1_SCK-Pad9) -> SCK
- C1 pad 1: +9V -> +5VD
- C16 pad 1: +5VD -> Net-(D3-K)
- C17 pad 1: +5VD -> Net-(D3-K)
- C3 pad 2: Net-(U2D-+) -> Net-(U2A-+)
- C5 pad 2: Net-(U2C-+) -> Net-(U2D-+)
- C7 pad 2: Net-(U2A-+) -> Net-(U2C-+)
- D2 pad 2: +5V -> +5VD
- J4 pad SN: unconnected-(J4-PadSN) -> GND
- J4 pad TN: unconnected-(J4-PadTN) -> AUDIO_IN_JACK_LEFT
- J5 pad SN: unconnected-(J5-PadSN) -> GND
- J5 pad TN: unconnected-(J5-PadTN) -> AUDIO_OUT_JACK_LEFT
- J7 pad SN: unconnected-(J7-PadSN) -> GND
- J7 pad TN: unconnected-(J7-PadTN) -> AUDIO_IN_JACK_RIGHT
- J8 pad SN: unconnected-(J8-PadSN) -> GND
- J8 pad TN: unconnected-(J8-PadTN) -> AUDIO_OUT_JACK_RIGHT
- R1 pad 1: Net-(U2A-+) -> Net-(U2C-+)
- R2 pad 1: Net-(U2C--) -> Net-(U2D--)
- R3 pad 1: Net-(U2D--) -> Net-(U2A--)
- U2 pad 1: AUDIO_IN_JACK_LEFT_BUF -> Net-(U2A--)
- U2 pad 2: AUDIO_IN_JACK_LEFT_BUF -> Net-(U2A--)
- U2 pad 8: Net-(U2C--) -> AUDIO_IN_JACK_LEFT_BUF
- U2 pad 9: Net-(U2C--) -> AUDIO_IN_JACK_LEFT_BUF
- U3 pad 1: GND -> Net-(U3-BOOT)
- U3 pad 2: +5VD -> unconnected-(U3-NC-Pad2)
- U3 pad 3: +9V -> unconnected-(U3-NC-Pad3)
Routing:
- net AUDIO_IN_JACK_RIGHT_BUF: track 0.00 -> 69.3 mm, vias 0 -> 2
- net AUDIO_IN_JACK_LEFT_BUF: track 0.00 -> 65.3 mm, vias 0 -> 2
- net Net-(U2A-+): track 0.00 -> 57.5 mm, vias 0 -> 2
- net +3.3VD: track 0.00 -> 52.7 mm
- net Net-(U2D-+): track 0.00 -> 51.7 mm, vias 0 -> 2
- net Net-(A1-I2C1_SCL): track 0.00 -> 50.3 mm
- net Net-(A1-I2C1_SDA): track 0.00 -> 50.3 mm
- net +9V: track 8.18 -> 55.4 mm, vias 0 -> 4
- net GND: track 0.00 -> 44.7 mm, vias 0 -> 23
- net PICO: track 0.00 -> 44.2 mm
- net POCI: track 0.00 -> 41.5 mm, vias 0 -> 1
- net SCK: track 0.00 -> 40.0 mm, vias 0 -> 1
- net AUDIO_IN_JACK_LEFT: track 0.00 -> 29.7 mm
- net Net-(A1-ADC_6): track 0.00 -> 27.7 mm
- net AUDIO_OUT_JACK_RIGHT: track 0.00 -> 27.6 mm
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- added copper zone on F.Cu, net +5VA
- added copper zone on In2.Cu, net +5VA
- added copper zone on F.Cu, net +5VD
- added copper zone on F.Cu, net +9V
- added copper zone on F.Cu, net GND
- added copper zone on In1.Cu, net GND
- added copper zone on F.Cu, net Net-(D6-K)
- added copper zone on F.Cu, net POWER_JACK_PWR
Other:
- board size 73 x 129 mm -> 73.5 x 129 mm
- board text added: "SCL"
- board text added: "SDA"

Commit message: tried to get SPI working
SPI drivers are thin on the esp-hal side and the ESP32 would not be able to initiate communication because of the master/slave setup, so I will try to get UART working.
Connections:
- A1 pad 8: GND -> CS
- U5 pad 8: GND -> CS
Changed lines of the file:
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@@
 			(layers "*.Cu" "*.Mask")
 			(remove_unused_layers no)
-			(net "GND")
+			(net "CS")
 			(pinfunction "SPI1_CS_8")
 			(pintype "bidirectional")
@@
 			(layers "*.Cu" "*.Mask")
 			(remove_unused_layers no)
-			(net "GND")
+			(net "CS")
 			(pinfunction "GPIO17_D7_RX_8")
 			(pintype "passive")
@@
 			(layers "F.Cu" "F.Mask")
 			(roundrect_rratio 0.1)
-			(net "GND")
+			(net "CS")
 			(pinfunction "GPIO17_D7_RX_8")
 			(pintype "passive")

Commit message: got pcb ready
Parts:
- moved C16 8.44 mm to (171.0, 157.8), turned to 180 degrees
- moved C17 7.84 mm to (171.0, 159.9), turned to 180 degrees
- moved J1 0.68 mm to (123.6, 100.8)
- moved R21 0.68 mm to (128.8, 103.2)
- moved R22 0.68 mm to (131.8, 103.2)
- moved J6 0.49 mm to (187.8, 129.8)
- moved A1 0.41 mm to (137.5, 157.8)
- moved R10 0.25 mm to (163.8, 59.8)
- moved C11 0.25 mm to (162.8, 70.5)
- moved C7 0.25 mm to (162.8, 57.3)
- moved D3 0.25 mm to (170.9, 153.2)
- moved R1 0.25 mm to (161.8, 59.8)
- moved R5 0.25 mm to (161.8, 68.0)
- moved R8 0.25 mm to (163.8, 68.0)
Connections:
- A1 pad 14: unconnected-(A1-USART1_TX-Pad14) -> DAISY_OUT
- A1 pad 15: unconnected-(A1-USART1_RX-Pad15) -> DAISY_IN
- U5 pad 5: unconnected-(U5-GPIO22_D4_SDA-Pad5) -> DAISY_OUT
- U5 pad 6: unconnected-(U5-GPIO23_D5_SCL-Pad6) -> DAISY_IN
Routing:
- net DAISY_OUT: track 0.00 -> 62.4 mm
- net DAISY_IN: track 0.00 -> 61.4 mm
- net CS: track 0.00 -> 39.2 mm
- net +9V: track 55.4 -> 44.8 mm, vias 4 -> 5
- net GND: track 44.7 -> 41.5 mm
- net AUDIO_IN_JACK_LEFT: track 29.7 -> 27.5 mm
- net AUDIO_IN_JACK_LEFT_BUF: track 65.3 -> 66.9 mm
- net +3.3VD: track 52.7 -> 54.2 mm
- net Net-(D3-K): track 7.60 -> 8.77 mm
- net Net-(U2D-+): track 51.7 -> 52.8 mm
- net Net-(A1-ADC_6): track 27.7 -> 28.5 mm
- net +5VD: track 15.6 -> 16.3 mm
- net AUDIO_OUT_JACK_RIGHT_BUF: track 2.65 -> 3.31 mm
- added copper zone on B.Cu, net +9V
Other:
- board size 73.5 x 129 mm -> 73.5 x 129.7 mm

Commit message: finished FFT sisplay test waiting for new PCB to arrive
Parts:
- A1: value Electrosmith_Daisy_Seed_Rev4 -> Electrosmith_Daisy_Seed_Rev4 (2 1x20 pin headers required)
- L1: footprint Inductor_SMD:L_6.3x6.3_H3 -> Inductor_SMD:L_Changjiang_FNR8040S
- U5: value XIAO-ESP32-C6-DIP -> XIAO-ESP32-C6-DIP (2 1x7 pin headers required)
- moved C17 10.8 mm to (180.5, 154.8), turned to 90 degrees
- moved C16 7.86 mm to (178.2, 154.8), turned to 90 degrees
- moved D3 6.78 mm to (168.2, 147.0), turned to -90 degrees
- moved L1 0.99 mm to (166.5, 155.0)
Routing:
- net PICO: track 44.0 -> 63.1 mm
- net +9V: track 44.8 -> 31.2 mm
- net Net-(D3-K): track 8.77 -> 20.9 mm
- net POCI: track 41.4 -> 50.6 mm, vias 1 -> 0
- net +5VD: track 16.3 -> 7.87 mm
- net GND: track 41.5 -> 36.2 mm, vias 23 -> 22
- net SCK: track 39.8 -> 41.8 mm
- net Net-(C6-Pad1): track 0.00 -> 1.70 mm
- net Net-(D6-K): track 0.00 -> 1.23 mm
- net CS: vias 0 -> 1

Commit message: pedal works but is buggy
Parts:
- removed the C15 at (150.6, 139.2)
- removed the J1 at (123.6, 100.8)
- removed the J6 at (187.8, 129.8)
- removed R21: 100, Resistor_SMD:R_0603_1608Metric
- removed R22: 10k, Resistor_SMD:R_0603_1608Metric
- removed R27: 1K, Resistor_SMD:R_0603_1608Metric
- added 5VA1: TestPoint, Connector_PinHeader_2.54mm:PinHeader_1x01_P2.54mm_Vertical, F.Cu at (152.8, 58.5)
- added 5VD1: TestPoint, Connector_PinHeader_2.54mm:PinHeader_1x01_P2.54mm_Vertical, F.Cu at (152.8, 54.8)
- added 9V1: TestPoint, Connector_PinHeader_2.54mm:PinHeader_1x01_P2.54mm_Vertical, F.Cu at (152.8, 62.2)
- added C12: 100uf, Capacitor_Tantalum_SMD:CP_EIA-3528-21_Kemet-B, F.Cu at (182.0, 49.0)
- added C16: 0.33uf, Capacitor_SMD:C_0805_2012Metric, F.Cu at (174.5, 55.0)
- added C17: 0.1uf, Capacitor_SMD:C_0805_2012Metric, F.Cu at (181.5, 55.0)
- added FB1: 120Ω@100MHz, Resistor_SMD:R_0603_1608Metric, F.Cu at (179.2, 52.2)
- added GND1: TestPoint, Connector_PinHeader_2.54mm:PinHeader_1x01_P2.54mm_Vertical, F.Cu at (198.2, 58.5)
- added J3: Screw_Terminal_01x02, TerminalBlock:TerminalBlock_Xinya_XY308-2.54-2P_1x02_P2.54mm_Horizontal, B.Cu at (199.7, 75.7)
- added R1: 100, Resistor_SMD:R_0603_1608Metric, F.Cu at (194.5, 77.8)
- added R16: 10k, Resistor_SMD:R_0603_1608Metric, F.Cu at (153.2, 51.0)
- added R2: 10k, Resistor_SMD:R_0603_1608Metric, F.Cu at (194.5, 79.2)
- A1, J4, J5: moved to B.Cu
- A2: renamed from U5; moved to B.Cu
- C18: value 10uf -> 0.1uf
- J1: renamed from J7; moved to B.Cu
- J2: renamed from J8; moved to B.Cu
- J6: renamed from J3; moved to B.Cu
- R14: renamed from R6; value 3.24k -> 3.3k
- moved D2 113.5 mm to (185.5, 48.8), turned to 90 degrees
- moved D3 112.1 mm to (171.5, 46.9), turned to 180 degrees
- moved C11 111.4 mm to (166.8, 46.8), turned to 90 degrees
- moved C13 107.3 mm to (179.2, 49.2)
- moved L1 105.6 mm to (161.2, 49.5), turned to -90 degrees
- moved J6 102.8 mm to (192.0, 56.0), turned to -90 degrees
- moved U2 102.6 mm to (169.7, 51.4), turned to 0 degrees
- moved J4 97.0 mm to (186.5, 141.6)
- moved R14 95.0 mm to (167.6, 55.0), turned to 0 degrees
- moved R13 94.7 mm to (164.4, 55.0), turned to 0 degrees
- moved U3 90.7 mm to (178.0, 56.0), turned to -90 degrees
- moved D4 90.5 mm to (155.8, 52.0)
- moved D1 89.6 mm to (159.7, 57.8), turned to 90 degrees
- moved C15 88.3 mm to (166.0, 58.3), turned to 0 degrees
- moved C1 81.5 mm to (156.2, 76.2), turned to 0 degrees
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- renumbered C16 to C1, C13 to C10, C20 to C11, C19 to C13, C1 to C15, C12 to C19, C17 to C2, C11 to C3, C7 to C4, C3 to C5, C9 to C6, C2 to C7, C5 to C8, C6 to C9, D3 to D1, D5 to D2, D6 to D3, D2 to D4, R4 to R10, R2 to R11, R11 to R12, R9 to R13, R23 to R15, R5 to R3, R8 to R4, R1 to R5, R10 to R6, R3 to R8, R12 to R9, U2 to U1, U3 to U2, U1 to U3
Connections:
- A1 pad 12: Net-(A1-I2C1_SCL) -> unconnected-(A1-I2C1_SCL-Pad12)
- A1 pad 13: Net-(A1-I2C1_SDA) -> unconnected-(A1-I2C1_SDA-Pad13)
- A1 pad 22: unconnected-(A1-ADC_0-Pad22) -> Net-(A1-ADC_0)
- A1 pad 28: Net-(A1-ADC_6) -> unconnected-(A1-ADC_6-Pad28)
- C14 pad 1: +5VA -> GND
- C14 pad 2: GND -> +9V
- C18 pad 1: GND -> +5VA
- C18 pad 2: +9V -> GND
- C3 pad 2: Net-(U2B-+) -> Net-(U1C-+)
- C4 pad 2: Net-(U2C-+) -> Net-(U1B-+)
- C5 pad 2: Net-(U2A-+) -> Net-(U1D-+)
- C8 pad 2: Net-(U2D-+) -> Net-(U1A-+)
- R11 pad 1: Net-(U2D--) -> Net-(U1A--)
- R3 pad 1: Net-(U2B-+) -> Net-(U1C-+)
- R5 pad 1: Net-(U2C-+) -> Net-(U1B-+)
- R8 pad 1: Net-(U2A--) -> Net-(U1D--)
- U1 pad 1: Net-(U2A--) -> Net-(U1A--)
- U1 pad 10: Net-(U2C-+) -> Net-(U1C-+)
- U1 pad 12: Net-(U2D-+) -> Net-(U1D-+)
- U1 pad 13: Net-(U2D--) -> Net-(U1D--)
- U1 pad 14: Net-(U2D--) -> Net-(U1D--)
- U1 pad 2: Net-(U2A--) -> Net-(U1A--)
- U1 pad 3: Net-(U2A-+) -> Net-(U1A-+)
- U1 pad 5: Net-(U2B-+) -> Net-(U1B-+)
- U1 pad 6: AUDIO_IN_JACK_RIGHT_BUF -> AUDIO_IN_JACK_LEFT_BUF
- U1 pad 7: AUDIO_IN_JACK_RIGHT_BUF -> AUDIO_IN_JACK_LEFT_BUF
- U1 pad 8: AUDIO_IN_JACK_LEFT_BUF -> AUDIO_IN_JACK_RIGHT_BUF
- U1 pad 9: AUDIO_IN_JACK_LEFT_BUF -> AUDIO_IN_JACK_RIGHT_BUF
- U3 pad 1: GND -> +5VA
- U3 pad 2: +5VA -> GND
- U3 pad 3: +9V -> Net-(U3-VI)
Routing:
- net Net-(U2A-+): track 57.5 -> 0.00 mm, vias 2 -> 0
- net +3.3VD: track 54.2 -> 0.00 mm
- net Net-(U2D-+): track 52.8 -> 0.00 mm, vias 2 -> 0
- net Net-(A1-I2C1_SCL): track 50.4 -> 0.00 mm
- net Net-(A1-I2C1_SDA): track 50.4 -> 0.00 mm
- net +9V: track 31.2 -> 80.6 mm, vias 5 -> 7
- net Net-(U1A-+): track 0.00 -> 47.4 mm, vias 0 -> 2
- net PICO: track 63.1 -> 21.7 mm
- net Net-(U1D-+): track 0.00 -> 38.3 mm, vias 0 -> 2
- net CS: track 39.2 -> 5.01 mm, vias 1 -> 0
- net POCI: track 50.6 -> 16.8 mm
- net SCK: track 41.8 -> 8.29 mm, vias 1 -> 0
- net DAISY_OUT: track 62.4 -> 29.5 mm
- net DAISY_IN: track 61.4 -> 29.5 mm
- net Net-(A1-ADC_0): track 0.00 -> 31.1 mm, vias 0 -> 1
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- added copper zone on In2.Cu, net +9V
- removed copper zone on F.Cu, net +5VA
- removed copper zone on B.Cu, net +9V
- removed copper zone on F.Cu, net POWER_JACK_PWR
Other:
- board size 73.5 x 129.7 mm -> 54 x 106 mm
- board text added: "5VA"
- board text added: "5VD"
- board text added: "9V"
- board text added: "GND"
- board text removed: "SCL"
- board text removed: "SDA"

Commit message: Update projects and ignore build output
Parts:
- removed C12: 100uf, Capacitor_Tantalum_SMD:CP_EIA-3528-21_Kemet-B
Changed lines of the file:
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@@
 		)
 	)
-	(footprint "Capacitor_Tantalum_SMD:CP_EIA-3528-21_Kemet-B"
-		(layer "F.Cu")
-		(at 182 49 90)
-		(descr "Tantalum Capacitor SMD Kemet-B (3528-21 Metric), IPC-7352 nominal, (Body size from: http://www.kemet.com/Lists/ProductCatalog/Attachments/253/KEM_TC101_STD.pdf)")
-		(tags "capacitor tantalum")
-		(property "Reference" "C12"
-			(at 4.25 0 180)
-			(layer "F.SilkS")
-			(effects
-				(font
-					(size 1 1)
-					(thickness 0.15)
-				)
-			)
-		)
-		(property "Value" "100uf"
-			(at 0 2.35 90)
-			(layer "F.Fab")
-			(effects
-				(font
-					(size 1 1)
-					(thickness 0.15)
-				)
-			)
-		)
-		(property "Datasheet" ""
-			(at 0 0 90)
-			(layer "F.Fab")
-			(hide yes)
-			(effects
-				(font
-					(size 1.27 1.27)
-				)
-			)
-		)
-		(property "Description" "Polarized capacitor"
-			(at 0 0 90)
-			(layer "F.Fab")
-			(hide yes)
-			(effects
-				(font
-					(size 1.27 1.27)
-				)
-			)
-		)
-		(property "KiLib_Generator" "SMD_2terminal_chip_molded"
-			(at 0 0 90)
-			(layer "F.SilkS")
-			(hide yes)
-			(effects
-				(font
-					(size 1 1)
-					(thickness 0.15)
-				)
-			)
-		)
-		(property "MPN" "C16133"
-			(at 0 0 90)
-			(unlocked yes)
-			(layer "F.Fab")
-			(hide yes)
-			(effects
-				(font
-					(size 1 1)
-					(thickness 0.15)
-				)
-			)
-		)
-		(property ki_fp_filters "CP_*")
-		(sheetname "/Power/")
-		(sheetfile "power.kicad_sch")
-		(units
-			(unit
-				(name "A")
-				(pins "1" "2")
-			)
-		)
-		(attr smd)
-		(duplicate_pad_numbers_are_jumpers no)
-		(fp_line
-			(start 1.75 -1.51)
-			(end -2.47 -1.51)
-			(stroke
-				(width 0.12)
-				(type solid)
-			)
-			(layer "F.SilkS")
-		)
-		(fp_line
-			(start -2.47 -1.51)
-			(end -2.47 1.51)
-			(stroke
-				(width 0.12)
-				(type solid)
-			)
-			(layer "F.SilkS")
-		)
-		(fp_line
-			(start -2.47 1.51)
-			(end 1.75 1.51)
-			(stroke
-				(width 0.12)
-				(type solid)
-			)
-			(layer "F.SilkS")
-		)
-		(fp_rect
-			(start -2.46 -1.65)
-			(end 2.46 1.65)
-			(stroke
-				(width 0.05)
-				(type solid)
-			)
-			(fill no)
-			(layer "F.CrtYd")
-		)
-		(fp_line
-			(start 1.75 -1.4)
-			(end -1.05 -1.4)
-			(stroke
-				(width 0.1)
-				(type solid)
-			)
-			(layer "F.Fab")
-		)
-		(fp_line
-			(start -1.05 -1.4)
-			(end -1.75 -0.7)
-			(stroke
-				(width 0.1)
-				(type solid)
-			)
-			(layer "F.Fab")
-		)
-		(fp_line
-			(start -1.75 -0.7)
-			(end -1.75 1.4)
-			(stroke
-				(width 0.1)
-				(type solid)
-			)
-			(layer "F.Fab")
-		)
-		(fp_line
-			(start 1.75 1.4)
-			(end 1.75 -1.4)
-			(stroke
-				(width 0.1)
-				(type solid)
-			)
-			(layer "F.Fab")
-		)
-		(fp_line
-			(start -1.75 1.4)
-			(end 1.75 1.4)
-			(stroke
-				(width 0.1)
-				(type solid)
-			)
-			(layer "F.Fab")
-		)
-		(fp_text user "${REFERENCE}"
-			(at 0 0 90)
-			(layer "F.Fab")
-			(effects
-				(font
-					(size 0.88 0.88)
-					(thickness 0.13)
-				)
-			)
-		)
-		(pad "1" smd roundrect
-			(at -1.54 0 90)
-			(size 1.34 2.39)
-			(layers "F.Cu" "F.Mask" "F.Paste")
-			(roundrect_rratio 0.186567)
-			(net "+9V")
-			(pintype "passive")
-		)
-		(pad "2" smd roundrect
-			(at 1.54 0 90)
-			(size 1.34 2.39)
-			(layers "F.Cu" "F.Mask" "F.Paste")
-			(roundrect_rratio 0.186567)
-			(net "GND")
-			(pintype "passive")
-		)
-		(embedded_fonts no)
-		(model "${KICAD10_3DMODEL_DIR}/Capacitor_Tantalum_SMD.3dshapes/CP_EIA-3528-21_Kemet-B.step"
-			(offset
-				(xyz 0 0 0)
-			)
-			(scale
-				(xyz 1 1 1)
-			)
-			(rotate
-				(xyz 0 0 0)
-			)
-		)
-	)
 	(footprint "Capacitor_SMD:C_0805_2012Metric"
 		(layer "F.Cu")
@@
 	)
 	(segment
+		(start 178.425 52.25)
+		(end 177.702978 52.25)
+		(width 1)
+		(layer "F.Cu")
+		(net "Net-(U3-VI)")
+	)
+	(segment
+		(start 174.5 54.05)
+		(end 174.32457 54.05)
+		(width 1)
+		(layer "F.Cu")
+		(net "Net-(U3-VI)")
+	)
+	(segment
+		(start 174.5 54.05)
+		(end 176.5 54.05)
+		(width 1)
+		(layer "F.Cu")
+		(net "Net-(U3-VI)")
+	)
+	(segment
+		(start 177.702978 52.25)
+		(end 176.5 53.452978)
+		(width 1)
+		(layer "F.Cu")
+		(net "Net-(U3-VI)")
+	)
+	(segment
+		(start 176.5 53.452978)
+		(end 176.5 54.05)
+		(width 1)
+		(layer "F.Cu")
+		(net "Net-(U3-VI)")
+	)
+	(segment
 		(start 153.668 76.25)
 		(end 153.418 76.5)
@@
 		(net "+3.3VA")
 	)
-	(segment
-		(start 178.425 52.25)
-		(end 177.702978 52.25)
-		(width 1)
-		(layer "F.Cu")
-		(net "Net-(U3-VI)")
-	)
-	(segment
-		(start 174.5 54.05)
-		(end 174.32457 54.05)
-		(width 1)
-		(layer "F.Cu")
-		(net "Net-(U3-VI)")
-	)
-	(segment
-		(start 174.5 54.05)
-		(end 176.5 54.05)
-		(width 1)
-		(layer "F.Cu")
-		(net "Net-(U3-VI)")
-	)
-	(segment
-		(start 177.702978 52.25)
-		(end 176.5 53.452978)
-		(width 1)
-		(layer "F.Cu")
-		(net "Net-(U3-VI)")
-	)
-	(segment
-		(start 176.5 53.452978)
-		(end 176.5 54.05)
-		(width 1)
-		(layer "F.Cu")
-		(net "Net-(U3-VI)")
-	)
 	(zone
