File: full-pcb/full_pcb.kicad_sch (KiCad schematic)
At the start: 23 parts, among them J1 Screw_Terminal_01x02, J4 AUDIO_IN_TRS, J5 AUDIO_OUT_TRS, J6 Screw_Terminal_01x02, P1 USB_C_Plug_USB2.0, U1 ESP32-C3-WROOM-02, U6 USBLC6-2SC6

Commit message: trouble with defmt
Parts:
- removed AUDIO_IN1, AUDIO_RAW1: TestPoint, TestPoint:TestPoint_Pad_D2.0mm, symbol Connector:TestPoint
- removed BOOT1, RESET1: SW_Push, Button_Switch_SMD:SW_SPST_TL3342, symbol Switch:SW_Push
- removed P1: USB_C_Plug_USB2.0, Connector_USB:USB_C_Receptacle_HRO_TYPE-C-31-M-17, symbol Connector:USB_C_Plug_USB2.0
- removed R15: 5.1k, Resistor_SMD:R_0603_1608Metric, symbol Device:R
- removed R24, R28, R29, R30: 10k, Resistor_SMD:R_0603_1608Metric, symbol Device:R
- removed U1: ESP32-C3-WROOM-02, RF_Module:ESP32-C3-WROOM-02, symbol RF_Module:ESP32-C3-WROOM-02
- removed U6: USBLC6-2SC6, Package_TO_SOT_SMD:SOT-23-6, symbol Power_Protection:USBLC6-2SC6
- added 5V2: TestPoint, TestPoint:TestPoint_Pad_D2.0mm, symbol Connector:TestPoint
- added D3: SS14, Diode_SMD:D_SMA, symbol Diode:1N5817
- added J7: AUDIO_IN_TRS, Connector_Audio:Jack_6.35mm_Neutrik_NMJ6HCD3_Horizontal, symbol NMJ6HCD2:NMJ6HCD2
- added J8: AUDIO_OUT_TRS, Connector_Audio:Jack_6.35mm_Neutrik_NMJ6HCD3_Horizontal, symbol NMJ6HCD2:NMJ6HCD2
- added U7: XIAO-ESP32-C3-DIP, Seeed Studio XIAO Series Library:XIAO-ESP32-C3-DIP, symbol Seeed_Studio_XIAO_Series:XIAO-ESP32-C3-DIP
Connections:
- net +3.3V: now also 5V2.1
- net AUDIO_IN_JACK_RIGHT: now also J7.T; no longer J4.R
- net AUDIO_OUT_JACK_RIGHT: now also J8.T; no longer J5.R
- net DAISY_IN: now also U7.7 (GPIO21_D6_TX)
- net DAISY_OUT: now also U7.8 (GPIO20_D7_RX)
- net GND: now also J7.S, J8.S, U7.13 (GND)
- new net: D3.1 (K), U7.14 (VBUS)
- new net +5VD: D3.2 (A)
- no-connect marks 34 -> 43
