File: full-pcb/full_pcb.kicad_sch (KiCad schematic)
At the start: 16 parts, among them J1 Screw_Terminal_01x02, J4 AUDIO_IN_TRS, J5 AUDIO_OUT_TRS, J6 Screw_Terminal_01x02, J7 AUDIO_IN_TRS, J8 AUDIO_OUT_TRS, U7 XIAO-ESP32-C3-DIP

Commit message: got the fft to work YAY!
Parts:
- removed 5V1, 5V2, 9V1, GND1, GND2: TestPoint, TestPoint:TestPoint_Pad_D2.0mm, symbol Connector:TestPoint
- removed U7: XIAO-ESP32-C3-DIP, Seeed Studio XIAO Series Library:XIAO-ESP32-C3-DIP, symbol Seeed_Studio_XIAO_Series:XIAO-ESP32-C3-DIP
- added C16, C17: 0.1uf, Capacitor_SMD:C_0805_2012Metric, symbol Device:C
- added U5: XIAO-ESP32-C6-DIP, Seeed Studio XIAO Series Library:XIAO-ESP32-C6-DIP, symbol Seeed_Studio_XIAO_Series:XIAO-ESP32-C6-DIP
Connections:
- net +3.3VD: now also A1.38 (3V3_D)
- net AUDIO_IN_JACK_LEFT: now also J4.TN
- net AUDIO_IN_JACK_RIGHT: now also J7.TN
- net AUDIO_OUT_JACK_LEFT: now also J5.TN
- net AUDIO_OUT_JACK_RIGHT: now also J8.TN
- net GND: now also A1.8 (SPI1_CS), J4.SN, J5.SN, J7.SN, J8.SN, C16.2, C17.2, U5.13 (GND), U5.8 (GPIO17_D7_RX)
- net at D3.1 (K): now also C16.1, C17.1, U5.14 (VBUS)
- net POCI: now reaches A1.10 (SPI1_POCI)
- net POCI: now also U5.10 (GPIO20_D9_MISO)
- net PICO: now reaches A1.11 (SPI1_PICO)
- net PICO: now also U5.11 (GPIO18_D10_MOSI)
- net SCK: now reaches A1.9 (SPI1_SCK)
- net SCK: now also U5.9 (GPIO19_D8_SCK)
- net DAISY_IN: no longer names the net of A1.15 (USART1_RX)
- net DAISY_OUT: no longer names the net of A1.14 (USART1_TX)
- no-connect marks 43 -> 40
Other:
- note added: "acts as CS pin"
- note added: "if using C3 be sure to use the XAIO board pins like A0_D0 and not the GPIO pins like GPIO0"
- moved on the sheet: D3

Commit message: tried to get SPI working
SPI drivers are thin on the esp-hal side and the ESP32 would not be able to initiate communication because of the master/slave setup, so I will try to get UART working.
Connections:
- net GND: no longer A1.8 (SPI1_CS), U5.8 (GPIO17_D7_RX)
- net DAISY_OUT: now reaches A1.14 (USART1_TX)
- net DAISY_OUT: now also U5.5 (GPIO22_D4_SDA)
- net DAISY_IN: now reaches A1.15 (USART1_RX)
- net DAISY_IN: now also U5.6 (GPIO23_D5_SCL)
- new net CS: A1.8 (SPI1_CS), U5.8 (GPIO17_D7_RX)
- no-connect marks 40 -> 36
Other:
- note removed: "acts as CS pin"
Changed lines of the file:
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@@
 		)
 	)
-	(text "acts as CS pin"
-		(exclude_from_sim no)
-		(at 268.986 122.174 0)
-		(effects
-			(font
-				(size 1.27 1.27)
-			)
-		)
-	)
 	(junction
 		(at -33.02 143.51)
@@
 	)
 	(no_connect
-		(at 214.63 114.3)
-	)
-	(no_connect
 		(at 119.38 123.19)
 	)
@@
 	)
 	(no_connect
+		(at 214.63 121.92)
+	)
+	(no_connect
 		(at 119.38 105.41)
 	)
@@
 	)
 	(no_connect
-		(at 170.18 85.09)
-	)
-	(no_connect
-		(at 214.63 121.92)
-	)
-	(no_connect
 		(at 46.99 137.16)
 	)
 	(no_connect
-		(at 170.18 82.55)
-	)
-	(no_connect
 		(at 214.63 106.68)
 	)
@@
 	)
 	(no_connect
-		(at 214.63 118.11)
-	)
-	(no_connect
 		(at 170.18 72.39)
 	)
@@
 		)
 	)
+	(global_label "CS"
+		(shape input)
+		(at 170.18 97.79 0)
+		(fields_autoplaced yes)
+		(effects
+			(font
+				(size 1.27 1.27)
+			)
+			(justify left)
+		)
+		(property "Intersheetrefs" "${INTERSHEET_REFS}"
+			(at 175.6447 97.79 0)
+			(hide yes)
+			(show_name no)
+			(do_not_autoplace no)
+			(effects
+				(font
+					(size 1.27 1.27)
+				)
+				(justify left)
+			)
+		)
+	)
+	(global_label "CS"
+		(shape input)
+		(at 252.73 121.92 0)
+		(fields_autoplaced yes)
+		(effects
+			(font
+				(size 1.27 1.27)
+			)
+			(justify left)
+		)
+		(property "Intersheetrefs" "${INTERSHEET_REFS}"
+			(at 258.1947 121.92 0)
+			(hide yes)
+			(show_name no)
+			(do_not_autoplace no)
+			(effects
+				(font
+					(size 1.27 1.27)
+				)
+				(justify left)
+			)
+		)
+	)
 	(global_label "AUDIO_OUT_JACK_LEFT_BUF"
 		(shape input)
@@
 		)
 	)
+	(global_label "DAISY_IN"
+		(shape input)
+		(at 214.63 118.11 180)
+		(fields_autoplaced yes)
+		(effects
+			(font
+				(size 1.27 1.27)
+			)
+			(justify right)
+		)
+		(property "Intersheetrefs" "${INTERSHEET_REFS}"
+			(at 203.4804 118.11 0)
+			(hide yes)
+			(show_name no)
+			(do_not_autoplace no)
+			(effects
+				(font
+					(size 1.27 1.27)
+				)
+				(justify right)
+			)
+		)
+	)
 	(global_label "SCK"
 		(shape input)
@@
 		)
 	)
+	(global_label "DAISY_OUT"
+		(shape input)
+		(at 170.18 82.55 0)
+		(fields_autoplaced yes)
+		(effects
+			(font
+				(size 1.27 1.27)
+			)
+			(justify left)
+		)
+		(property "Intersheetrefs" "${INTERSHEET_REFS}"
+			(at 183.0229 82.55 0)
+			(hide yes)
+			(show_name no)
+			(do_not_autoplace no)
+			(effects
+				(font
+					(size 1.27 1.27)
+				)
+				(justify left)
+			)
+		)
+	)
 	(global_label "AUDIO_OUT_JACK_RIGHT"
 		(shape input)
@@
 		)
 	)
+	(global_label "DAISY_IN"
+		(shape input)
+		(at 170.18 85.09 0)
+		(fields_autoplaced yes)
+		(effects
+			(font
+				(size 1.27 1.27)
+			)
+			(justify left)
+		)
+		(property "Intersheetrefs" "${INTERSHEET_REFS}"
+			(at 181.3296 85.09 0)
+			(hide yes)
+			(show_name no)
+			(do_not_autoplace no)
+			(effects
+				(font
+					(size 1.27 1.27)
+				)
+				(justify left)
+			)
+		)
+	)
+	(global_label "DAISY_OUT"
+		(shape input)
+		(at 214.63 114.3 180)
+		(fields_autoplaced yes)
+		(effects
+			(font
+				(size 1.27 1.27)
+			)
+			(justify right)
+		)
+		(property "Intersheetrefs" "${INTERSHEET_REFS}"
+			(at 201.7871 114.3 0)
+			(hide yes)
+			(show_name no)
+			(do_not_autoplace no)
+			(effects
+				(font
+					(size 1.27 1.27)
+				)
+				(justify right)
+			)
+		)
+	)
 	(global_label "AUDIO_OUT_JACK_RIGHT_BUF"
 		(shape input)
@@
 	)
 	(symbol
-		(lib_id "power:GNDA")
-		(at 252.73 121.92 90)
-		(unit 1)
-		(body_style 1)
-		(exclude_from_sim no)
-		(in_bom yes)
-		(on_board yes)
-		(in_pos_files yes)
-		(dnp no)
-		(fields_autoplaced yes)
-		(property "Reference" "#PWR029"
-			(at 259.08 121.92 0)
-			(hide yes)
-			(show_name no)
-			(do_not_autoplace no)
-			(effects
-				(font
-					(size 1.27 1.27)
-				)
-			)
-		)
-		(property "Value" "GND"
-			(at 256.54 121.9199 90)
-			(show_name no)
-			(do_not_autoplace no)
-			(effects
-				(font
-					(size 1.27 1.27)
-				)
-				(justify right)
-			)
-		)
-		(property "Footprint" ""
-			(at 252.73 121.92 0)
-			(hide yes)
-			(show_name no)
-			(do_not_autoplace no)
-			(effects
-				(font
-					(size 1.27 1.27)
-				)
-			)
-		)
-		(property "Datasheet" ""
-			(at 252.73 121.92 0)
-			(hide yes)
-			(show_name no)
-			(do_not_autoplace no)
-			(effects
-				(font
-					(size 1.27 1.27)
-				)
-			)
-		)
-		(property "Description" "Power symbol creates a global label with name \"GNDA\" , analog ground"
-			(at 252.73 121.92 0)
-			(hide yes)
-			(show_name no)
-			(do_not_autoplace no)
-			(effects
-				(font
-					(size 1.27 1.27)
-				)
-			)
-		)
-		(pin "1"
-		)
-		(instances
-			(project "full_pcb"
-				(path "/ac8ee366-0662-41f8-9745-078ec3fbb21b"
-					(reference "#PWR029")
-					(unit 1)
-				)
-			)
-		)
-	)
-	(symbol
 		(lib_id "Connector:Screw_Terminal_01x02")
 		(at 83.82 105.41 180)
@@
 					(unit 1)
 				)
-			)
-		)
-	)
-	(symbol
-		(lib_id "power:GNDA")
-		(at 170.18 97.79 90)
-		(unit 1)
-		(body_style 1)
-		(exclude_from_sim no)
-		(in_bom yes)
-		(on_board yes)
-		(in_pos_files yes)
-		(dnp no)
-		(fields_autoplaced yes)
-		(property "Reference" "#PWR030"
-			(at 176.53 97.79 0)
-			(hide yes)
-			(show_name no)
-			(do_not_autoplace no)
-			(effects
-				(font
-					(size 1.27 1.27)
-				)
-			)
-		)
-		(property "Value" "GND"
-			(at 173.99 97.7899 90)
-			(show_name no)
-			(do_not_autoplace no)
-			(effects
-				(font
-					(size 1.27 1.27)
-				)
-				(justify right)
-			)
-		)
-		(property "Footprint" ""
-			(at 170.18 97.79 0)
-			(hide yes)
-			(show_name no)
-			(do_not_autoplace no)
-			(effects
-				(font
-					(size 1.27 1.27)
-				)
-			)
-		)
-		(property "Datasheet" ""
-			(at 170.18 97.79 0)
-			(hide yes)
-			(show_name no)
-			(do_not_autoplace no)
-			(effects
-				(font
-					(size 1.27 1.27)
-				)
-			)
-		)
-		(property "Description" "Power symbol creates a global label with name \"GNDA\" , analog ground"
-			(at 170.18 97.79 0)
-			(hide yes)
-			(show_name no)
-			(do_not_autoplace no)
-			(effects
-				(font
-					(size 1.27 1.27)
-				)
-			)
-		)
-		(pin "1"
-		)
-		(instances
-			(project "full_pcb"
-				(path "/ac8ee366-0662-41f8-9745-078ec3fbb21b"
-					(reference "#PWR030")
-					(unit 1)
-				)

Commit message: finished FFT sisplay test waiting for new PCB to arrive
Parts:
- A1: value Electrosmith_Daisy_Seed_Rev4 -> Electrosmith_Daisy_Seed_Rev4 (2 1x20 pin headers required); now left out of the parts list
- J4, J5, J7, J8: MPN (none) -> C368502
- U5: value XIAO-ESP32-C6-DIP -> XIAO-ESP32-C6-DIP (2 1x7 pin headers required); MPN (none) -> C5371993; now left out of the parts list
Other:
- note added: "if not using C6 be sure to use the XAIO board pins like A0_D0 and not the GPIO pins like GPIO0"
- note removed: "if using C3 be sure to use the XAIO board pins like A0_D0 and not the GPIO pins like GPIO0"
- moved on the sheet: J7, J8

Commit message: pedal works but is buggy
Parts:
- removed J1, J6: Screw_Terminal_01x02, TerminalBlock:TerminalBlock_Xinya_XY308-2.54-2P_1x02_P2.54mm_Horizontal, symbol Connector:Screw_Terminal_01x02
- removed R21: 100, Resistor_SMD:R_0603_1608Metric, symbol Device:R
- removed R22: 10k, Resistor_SMD:R_0603_1608Metric, symbol Device:R
- added J3: Screw_Terminal_01x02, TerminalBlock:TerminalBlock_Xinya_XY308-2.54-2P_1x02_P2.54mm_Horizontal, symbol Connector:Screw_Terminal_01x02
- added R1: 100, Resistor_SMD:R_0603_1608Metric, symbol Device:R
- added R2: 10k, Resistor_SMD:R_0603_1608Metric, symbol Device:R
- A1: now in the parts list
- A2: renamed from U5; now in the parts list
- J1: renamed from J7; now not fitted; now left out of the parts list
- J2: renamed from J8; now not fitted; now left out of the parts list
- J4, J5: now not fitted; now left out of the parts list
- renumbered C16 to C1, C17 to C2, D3 to D1
Connections:
- net +3.3VA: now also J3.1 (Pin_1)
- net GND: now also R2.2
- net at A1.22 (ADC_0): now also R1.1, R2.1
- new net: J3.2 (Pin_2), R1.2
- no-connect marks 36 -> 38
