File: full-pcb/power.kicad_sch (KiCad schematic)
At the start: 19 parts, among them J3 Barrel_Jack_Switch, U2 OPA1664D, U3 AMS1117-5.0, U4 CJ431, U5 AMS1117-3.3

Commit message: trouble with defmt
Parts:
- removed C15, C19: 10uf, Capacitor_Tantalum_SMD:CP_EIA-3216-18_Kemet-A, symbol Device:C_Polarized
- removed C20: 0.1uf, Capacitor_SMD:C_0805_2012Metric, symbol Device:C
- removed U5: AMS1117-3.3, Package_TO_SOT_SMD:SOT-223-3_TabPin2, symbol Regulator_Linear:LM1117DT-5.0
- added C15: 10uf, Capacitor_SMD:C_0805_2012Metric, symbol Device:C
- added C16, C17: 0.1uf, Capacitor_SMD:C_0805_2012Metric, symbol Device:C
- added U1: 78L05G-AB3-R, Package_TO_SOT_SMD:SOT-89-3, symbol Regulator_Linear:AZ1117R-ADJ
- C14: value 10uf -> 0.1uf; MPN C440198 -> C49678
- C18: value 0.1uf -> 10uf; MPN C49678 -> C440198
- D1: value 1N5817 -> SS34; footprint Diode_SMD:D_SOD-123 -> Diode_SMD:D_SMA; MPN C8598 -> C8678
- R27: value 330 -> 1K; MPN C23138 -> C21190
Connections:
- net +5V: no longer C10.1, C12.1, C14.2, C4.1, R23.2, U2.4 (V+), U3.2 (VO)
- net +9V: now also C18.2, U1.3 (VI); no longer C18.1
- net GND: now also C14.2, C18.1, C15.1, C16.2, C17.2, U1.1 (ADJ); no longer C14.1, C18.2
- new net +5VA: C12.1, C14.1, C15.2, R23.2, U1.2 (VO), U2.4 (V+)
- new net +5VD: C10.1, C16.1, C17.1, C4.1, U3.2 (VO)
