File: full-pcb/power.kicad_sch (KiCad schematic)
At the start: 19 parts, among them J3 Barrel_Jack_Switch, U1 78L05G-AB3-R, U2 OPA1664D, U3 AMS1117-5.0, U4 CJ431

Commit message: got the fft to work YAY!
Parts:
- removed C10, C16, C17, C8: 0.1uf, Capacitor_SMD:C_0805_2012Metric, symbol Device:C
- removed C4: 10uf, Capacitor_Tantalum_SMD:CP_EIA-3216-18_Kemet-A, symbol Device:C_Polarized
- removed D1: SS34, Diode_SMD:D_SMA, symbol Diode:1N5817
- removed U3: AMS1117-5.0, Package_TO_SOT_SMD:SOT-223-3_TabPin2, symbol Regulator_Linear:LM1117DT-5.0
- added C19: 10uf, Capacitor_SMD:C_0805_2012Metric, symbol Device:C
- added C20: 0.01uf, Capacitor_SMD:C_0805_2012Metric, symbol Device:C
- added D5, D6: SS34, Diode_SMD:D_SMA, symbol Diode:1N5817
- added L1: 18uH, Inductor_SMD:L_6.3x6.3_H3, symbol Device:L
- added R6: 3.24k, Resistor_SMD:R_0603_1608Metric, symbol Device:R
- added R9: 10k, Resistor_SMD:R_0603_1608Metric, symbol Device:R
- added U3: TPS5430DDA, Package_SO:TI_SO-PowerPAD-8_ThermalVias, symbol Regulator_Switching:TPS5430DDA
- C1: value 10uf -> 220uf; footprint Capacitor_Tantalum_SMD:CP_EIA-3216-18_Kemet-A -> Capacitor_Tantalum_SMD:CP_EIA-7343-31_Kemet-D; MPN C7171 -> C242173
- U4: MPN C21190 -> C3113
Connections:
- net +5V is gone; now on net +5VD: D2.2 (A)
- net +5VD: now also C1.1, L1.2, R9.1
- net +9V: now also C19.2, D5.1 (K), U3.7 (VIN); no longer C1.1
- net GND: now also C19.1, D6.2 (A), R6.2, U3.6 (GND), U3.9 (GNDPAD)
- net POWER_JACK_PWR: now also D5.2 (A)
- new net: C20.1, U3.1 (BOOT)
- new net: C20.2, D6.1 (K), L1.1, U3.8 (PH)
- new net: R6.1, R9.2, U3.4 (VSENSE)

Commit message: finished FFT sisplay test waiting for new PCB to arrive
Parts:
- L1: footprint Inductor_SMD:L_6.3x6.3_H3 -> Inductor_SMD:L_Changjiang_FNR8040S; MPN C20612510 -> C168130
Changed lines of the file:
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@@
 			)
 		)
-		(property "Footprint" "Inductor_SMD:L_6.3x6.3_H3"
+		(property "Footprint" "Inductor_SMD:L_Changjiang_FNR8040S"
 			(at 209.55 72.39 0)
 			(hide yes)
@@
 			)
 		)
-		(property "Datasheet" ""
+		(property "Datasheet" "C168130"
 			(at 209.55 72.39 0)
 			(hide yes)
@@
 			)
 		)
-		(property "MPN" "C20612510"
+		(property "MPN" "C168130"
 			(at 209.55 72.39 90)
 			(hide yes)

Commit message: pedal works but is buggy
Parts:
- removed C15: 10uf, Capacitor_SMD:C_0805_2012Metric, symbol Device:C
- removed R27: 1K, Resistor_SMD:R_0603_1608Metric, symbol Device:R
- added 5VA1, 5VD1, 9V1, GND1: TestPoint, Connector_PinHeader_2.54mm:PinHeader_1x01_P2.54mm_Vertical, symbol Connector:TestPoint
- added C12: 100uf, Capacitor_Tantalum_SMD:CP_EIA-3528-21_Kemet-B, symbol Device:C_Polarized
- added C16: 0.33uf, Capacitor_SMD:C_0805_2012Metric, symbol Device:C
- added C17: 0.1uf, Capacitor_SMD:C_0805_2012Metric, symbol Device:C
- added FB1: 120Ω@100MHz, Resistor_SMD:R_0603_1608Metric, symbol Device:FerriteBead
- added R16: 10k, Resistor_SMD:R_0603_1608Metric, symbol Device:R
- C18: value 10uf -> 0.1uf; MPN C440198 -> C49678
- R14: renamed from R6; value 3.24k -> 3.3k; MPN C166817 -> C22978
- U2: renamed from U3; MPN (none) -> C9864
- renumbered C20 to C11, C19 to C13, C1 to C15, C12 to C19, D5 to D2, D6 to D3, D2 to D4, J3 to J6, R9 to R13, R23 to R15, U2 to U1, U1 to U3
Connections:
- net +5VA: now also C18.1, U3.1 (VO), 5VA1.1, C17.2; no longer C14.1, U3.2 (VO)
- net +5VD: now also 5VD1.1
- net +9V: now also C14.2, 9V1.1, C12.1, FB1.1; no longer C18.2, U3.3 (VI)
- net GND: now also C14.1, C18.2, U3.2 (GND), C12.2, C16.1, C17.1, GND1.1, R16.1; no longer C14.2, C18.1, U3.1 (ADJ)
- net at D4.1 (K): now also R16.2
- new net: C16.2, FB1.2, U3.3 (VI)
- no-connect marks 0 -> 1
Other:
- moved on the sheet: C11, C13, C15, C19, D2, D3, D4, J6, L1, R13, R14, R15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

Commit message: updated pictures
Parts:
- removed C12: 100uf, Capacitor_Tantalum_SMD:CP_EIA-3528-21_Kemet-B, symbol Device:C_Polarized
Changed lines of the file:
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@@
 	)
 	(junction
-		(at 52.07 31.75)
-		(diameter 0)
-		(color 0 0 0 0)
-	)
-	(junction
 		(at 116.84 90.17)
 		(diameter 0)
@@
 	(wire
 		(pts
-			(xy 52.07 31.75) (xy 58.42 31.75)
-		)
-		(stroke
-			(width 0)
-			(type default)
-		)
-	)
-	(wire
-		(pts
 			(xy 132.08 31.75) (xy 137.16 31.75)
 		)
@@
 	(wire
 		(pts
-			(xy 45.72 31.75) (xy 52.07 31.75)
+			(xy 45.72 31.75) (xy 58.42 31.75)
 		)
 		(stroke
@@
 	)
 	(symbol
-		(lib_id "Device:C_Polarized")
-		(at 52.07 35.56 0)
-		(unit 1)
-		(body_style 1)
-		(exclude_from_sim no)
-		(in_bom yes)
-		(on_board yes)
-		(in_pos_files yes)
-		(dnp no)
-		(property "Reference" "C12"
-			(at 42.418 35.56 0)
-			(show_name no)
-			(do_not_autoplace no)
-			(effects
-				(font
-					(size 1.27 1.27)
-				)
-				(justify left)
-			)
-		)
-		(property "Value" "100uf"
-			(at 42.418 38.1 0)
-			(show_name no)
-			(do_not_autoplace no)
-			(effects
-				(font
-					(size 1.27 1.27)
-				)
-				(justify left)
-			)
-		)
-		(property "Footprint" "Capacitor_Tantalum_SMD:CP_EIA-3528-21_Kemet-B"
-			(at 53.0352 39.37 0)
-			(hide yes)
-			(show_name no)
-			(do_not_autoplace no)
-			(effects
-				(font
-					(size 1.27 1.27)
-				)
-			)
-		)
-		(property "Datasheet" ""
-			(at 52.07 35.56 0)
-			(hide yes)
-			(show_name no)
-			(do_not_autoplace no)
-			(effects
-				(font
-					(size 1.27 1.27)
-				)
-			)
-		)
-		(property "Description" "Polarized capacitor"
-			(at 52.07 35.56 0)
-			(hide yes)
-			(show_name no)
-			(do_not_autoplace no)
-			(effects
-				(font
-					(size 1.27 1.27)
-				)
-			)
-		)
-		(property "MPN" "C16133"
-			(at 52.07 35.56 0)
-			(hide yes)
-			(show_name no)
-			(do_not_autoplace no)
-			(effects
-				(font
-					(size 1.27 1.27)
-				)
-			)
-		)
-		(pin "2"
-		)
-		(pin "1"
-		)
-		(instances
-			(project "full_pcb"
-				(path "/ac8ee366-0662-41f8-9745-078ec3fbb21b/ecf25a48-7940-4cdf-9049-43d792c69dfb"
-					(reference "C12")
-					(unit 1)
-				)
-			)
-		)
-	)
-	(symbol
 		(lib_id "Device:C")
 		(at 83.82 35.56 180)
@@
 					(unit 1)
 				)
-			)
-		)
-	)
-	(symbol
-		(lib_name "GND_1")
-		(lib_id "power:GND")
-		(at 52.07 39.37 0)
-		(unit 1)
-		(body_style 1)
-		(exclude_from_sim no)
-		(in_bom yes)
-		(on_board yes)
-		(in_pos_files yes)
-		(dnp no)
-		(fields_autoplaced yes)
-		(property "Reference" "#PWR029"
-			(at 52.07 45.72 0)
-			(hide yes)
-			(show_name no)
-			(do_not_autoplace no)
-			(effects
-				(font
-					(size 1.27 1.27)
-				)
-			)
-		)
-		(property "Value" "GND"
-			(at 52.07 44.45 0)
-			(show_name no)
-			(do_not_autoplace no)
-			(effects
-				(font
-					(size 1.27 1.27)
-				)
-			)
-		)
-		(property "Footprint" ""
-			(at 52.07 39.37 0)
-			(hide yes)
-			(show_name no)
-			(do_not_autoplace no)
-			(effects
-				(font
-					(size 1.27 1.27)
-				)
-			)
-		)
-		(property "Datasheet" ""
-			(at 52.07 39.37 0)
-			(hide yes)
-			(show_name no)
-			(do_not_autoplace no)
-			(effects
-				(font
-					(size 1.27 1.27)
-				)
-			)
-		)
-		(property "Description" "Power symbol creates a global label with name \"GND\" , ground"
-			(at 52.07 39.37 0)
-			(hide yes)
-			(show_name no)
-			(do_not_autoplace no)
-			(effects
-				(font
-					(size 1.27 1.27)
-				)
-			)
-		)
-		(pin "1"
-		)
-		(instances
-			(project "full_pcb"
-				(path "/ac8ee366-0662-41f8-9745-078ec3fbb21b/ecf25a48-7940-4cdf-9049-43d792c69dfb"
-					(reference "#PWR029")
-					(unit 1)
-				)
