File: seed-pedal/Input.kicad_sch (KiCad schematic)
At the start: 27 parts, among them U1 OPA1654

Commit message: Update projects and ignore build output
Parts:
- removed R15, R8: 10k, Resistor_SMD:R_0603_1608Metric, symbol Device:R
- renumbered R11 to R10, R12 to R11, R13 to R12, R14 to R13, R16 to R14, R9 to R8, R10 to R9
