File: seed-pedal/power.kicad_sch (KiCad schematic)
At the start: 31 parts, among them J6 Barrel_Jack_Switch, U3 AMS1117-5.0, U4 OPA1652

Commit message: Update projects and ignore build output
Parts:
- removed C27, C28: 100uf, Capacitor_Tantalum_SMD:CP_EIA-3528-21_Kemet-B, symbol Device:C_Polarized
- removed C31: 10uf, Capacitor_Tantalum_SMD:CP_EIA-3216-18_Kemet-A, symbol Device:C_Polarized
- removed R28, R33, R34: 2.2, Resistor_SMD:R_0805_2012Metric, symbol Device:R
- removed R39: 10k, Resistor_SMD:R_0603_1608Metric, symbol Device:R
- removed U4: OPA1652, Package_SO:SOIC-8_3.9x4.9mm_P1.27mm, symbol Amplifier_Operational:OPA1656ID
- added C27: 10uf, Capacitor_SMD:C_0805_2012Metric, symbol Device:C
- added Q1, Q2: NPN, Package_TO_SOT_SMD:SOT-89-3, symbol Simulation_SPICE:NPN
- added R24: 1k, Resistor_SMD:R_0603_1608Metric, symbol Device:R
- C22, C24, C25: footprint Capacitor_Tantalum_SMD:CP_EIA-3528-21_Kemet-B -> Capacitor_THT:CP_Radial_D8.0mm_P3.50mm; MPN C16133 -> C5113358; now left out of the parts list
- C30: renamed from C34; footprint Capacitor_Tantalum_SMD:CP_EIA-3528-21_Kemet-B -> Capacitor_THT:CP_Radial_D8.0mm_P3.50mm; MPN C16133 -> C5113358; now left out of the parts list
- R23: renamed from R27; value 2.2 -> 1k; footprint Resistor_SMD:R_0805_2012Metric -> Resistor_SMD:R_0603_1608Metric; MPN C17521 -> C21190
- renumbered C30 to C26, C32 to C28, C33 to C29, R37 to R25, R38 to R26
Connections:
- net +9V: now also Q1.1 (C), Q2.1 (C), R24.1; no longer C21.2, C22.2, C23.2, C24.2, C25.2, C26.2, C28.2, C29.2, C30.2, GND1.1, J6.1, J6.3, R25.2, R26.1, U3.1 (GND)
- net ADUIO_VREF: now also C28.1, C29.1, C30.1, R25.1, R26.2
- net DAISY_POWER: now also Q1.3 (E); no longer C25.1
- net ESP_POWER: now also C27.2
- net at C24.1, R23.2: now also Q1.2 (B)
- new net: C25.1, Q2.2 (B), R24.2
- new net +9VA: Q2.3 (E), R25.2
- new net GND: C21.2, C22.2, C23.2, C24.2, C25.2, C26.2, C27.1, C28.2, C29.2, C30.2, GND1.1, J6.1, J6.3, R26.1, U3.1 (GND)
Other:
- note removed: "200mA limit"
- moved on the sheet: R23

Commit message: updated pictures
Parts:
- added U4: LM358, Package_SO:SOIC-8_3.9x4.9mm_P1.27mm, symbol Amplifier_Operational:LM358
Connections:
- net +9VA: now also U4.8 (V+)
- net ADUIO_VREF: now also U4.1, U4.2 (-); no longer C28.1, C29.1, C30.1, R25.1, R26.2
- net GND: now also U4.4 (V-), U4.5 (+)
- new net: U4.6 (-), U4.7
- new net: C28.1, C29.1, C30.1, R25.1, R26.2, U4.3 (+)
