File: seed-pedal/seed-pedal.kicad_pcb (KiCad board)
At the start: 4 copper layers, 54 x 106 mm, 82 parts, among them J1 AUDIO_IN_TRS, J2 AUDIO_OUT_TRS, J3 Screw_Terminal_01x02, J4 AUDIO_IN_TRS, J5 AUDIO_OUT_TRS, J6 Barrel_Jack_Switch, U1 OPA1654, U2 OPA1652, U3 AMS1117-5.0, U4 OPA1652

Commit message: Update projects and ignore build output
Parts:
- removed C31: 10uf, Capacitor_Tantalum_SMD:CP_EIA-3216-18_Kemet-A
- removed C32: 0.1uf, Capacitor_SMD:C_0805_2012Metric
- removed C33: 1uf, Capacitor_SMD:C_0805_2012Metric
- removed C34: 100uf, Capacitor_Tantalum_SMD:CP_EIA-3528-21_Kemet-B
- removed the R17 at (152.7, 93.0)
- removed R27, R28, R33, R34: 2.2, Resistor_SMD:R_0805_2012Metric
- removed R37, R38, R39: 10k, Resistor_SMD:R_0603_1608Metric
- removed the R9 at (157.4, 115.2)
- removed U4: OPA1652, Package_SO:SOIC-8_3.9x4.9mm_P1.27mm
- added C29: 1uf, Capacitor_SMD:C_0805_2012Metric, F.Cu at (155.5, 57.2)
- added C30: 100uf, Capacitor_THT:CP_Radial_D8.0mm_P3.50mm, B.Cu at (152.1, 55.2)
- added Q1: NPN, Package_TO_SOT_SMD:SOT-89-3, F.Cu at (136.8, 59.0)
- added Q2: NPN, Package_TO_SOT_SMD:SOT-89-3, F.Cu at (144.8, 58.9)
- added R23: 1k, Resistor_SMD:R_0603_1608Metric, F.Cu at (132.9, 58.3)
- added R24: 1k, Resistor_SMD:R_0603_1608Metric, F.Cu at (141.1, 58.2)
- added R25: 10k, Resistor_SMD:R_0603_1608Metric, F.Cu at (152.2, 59.0)
- added R26: 10k, Resistor_SMD:R_0603_1608Metric, F.Cu at (152.2, 57.5)
- C22, C24, C25: footprint Capacitor_Tantalum_SMD:CP_EIA-3528-21_Kemet-B -> Capacitor_THT:CP_Radial_D8.0mm_P3.50mm; moved to B.Cu
- C27: value 100uf -> 10uf; footprint Capacitor_Tantalum_SMD:CP_EIA-3528-21_Kemet-B -> Capacitor_SMD:C_0805_2012Metric
- C28: value 100uf -> 0.1uf; footprint Capacitor_Tantalum_SMD:CP_EIA-3528-21_Kemet-B -> Capacitor_SMD:C_0805_2012Metric
- R15: value 10k -> 33k
- R8: value 10k -> 1M
- moved R16 40.0 mm to (152.8, 96.0), turned to 180 degrees
- moved R15 39.8 mm to (152.8, 93.0), turned to 0 degrees
- moved R20 29.0 mm to (163.3, 95.1)
- moved C27 25.6 mm to (145.2, 76.0), turned to 90 degrees
- moved C24 23.9 mm to (134.8, 55.2), turned to 0 degrees
- moved C25 22.3 mm to (143.4, 55.2), turned to 0 degrees
- moved U3 15.6 mm to (139.5, 74.5)
- moved D1 14.9 mm to (133.2, 74.5), turned to 90 degrees
- moved C26 13.8 mm to (145.2, 72.8)
- moved C28 13.7 mm to (155.5, 59.2), turned to 0 degrees
- moved C23 12.1 mm to (162.5, 53.0), turned to 0 degrees
- moved C22 9.89 mm to (160.7, 55.2), turned to 0 degrees
- moved D2 8.01 mm to (157.2, 50.2), turned to 0 degrees
- moved C21 6.65 mm to (169.2, 52.8)
- moved FB1 6.20 mm to (168.8, 50.0)
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- renumbered C30 to C26, R11 to R10, R12 to R11, R13 to R12, R14 to R13, R16 to R14, R18 to R16, R19 to R17, R20 to R18, R21 to R19, R22 to R20, R23 to R21, R24 to R22, R10 to R9
Connections:
- C25 pad 1: DAISY_POWER -> Net-(Q2-B)
- C27 pad 1: Net-(C27-Pad1) -> GND
- C27 pad 2: GND -> ESP_POWER
- C28 pad 1: +9VA -> ADUIO_VREF
- R15 pad 1: GND -> Net-(C15-Pad2)
- R15 pad 2: AUDIO_IN_JACK_LEFT -> Net-(U2A-+)
- R8 pad 1: GND -> ADUIO_VREF
- R8 pad 2: AUDIO_IN_JACK_RIGHT -> Net-(C4-Pad2)
Routing:
- net ADUIO_VREF: track 1.18 -> 93.5 mm, vias 1 -> 5
- net AUDIO_IN_JACK_LEFT_BUF: track 1.52 -> 65.9 mm
- net AUDIO_OUT_JACK_LEFT: track 0.00 -> 58.9 mm
- net AUDIO_IN_JACK_RIGHT_BUF: track 0.00 -> 36.6 mm
- net AUDIO_OUT_JACK_RIGHT_BUF: track 0.00 -> 33.6 mm, vias 0 -> 1
- net AUDIO_OUT_JACK_RIGHT: track 0.50 -> 31.8 mm
- net AUDIO_IN_JACK_RIGHT: track 0.55 -> 29.9 mm
- net Net-(A1-ADC_0): track 0.00 -> 28.6 mm
- net AUDIO_IN_JACK_LEFT: track 1.52 -> 30.1 mm
- net +3.3VA: track 0.00 -> 27.5 mm
- net +9V: track 0.00 -> 25.9 mm, vias 0 -> 26
- net DAISY_POWER: track 68.4 -> 43.5 mm, vias 0 -> 1
- net Net-(A2-VBUS): track 28.1 -> 8.03 mm
- net GND: track 25.8 -> 42.6 mm, vias 9 -> 18
- net AUDIO_OUT_JACK_LEFT_BUF: track 0.00 -> 16.6 mm, vias 0 -> 1
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- added copper zone on In2.Cu, net +9V
- added copper zone on F.Cu, net ADUIO_VREF
- added copper zone on F.Cu, net Net-(C21-Pad1)
- removed copper zone on F.Cu, net Net-(C20-Pad1)
- removed copper zone on F.Cu, net Net-(D2-A)

Commit message: updated pictures
Parts:
- added U4: LM358, Package_SO:SOIC-8_3.9x4.9mm_P1.27mm, F.Cu at (162.5, 59.0)
Connections:
- C28 pad 1: ADUIO_VREF -> Net-(U4A-+)
- C29 pad 1: ADUIO_VREF -> Net-(U4A-+)
- C30 pad 1: ADUIO_VREF -> Net-(U4A-+)
- R25 pad 1: ADUIO_VREF -> Net-(U4A-+)
- R26 pad 2: ADUIO_VREF -> Net-(U4A-+)
Routing:
- net +9VA: track 89.3 -> 104.3 mm, vias 3 -> 4
- net Net-(U4A-+): track 0.00 -> 8.82 mm
- net ADUIO_VREF: track 93.5 -> 97.8 mm
- added copper zone on F.Cu, net Net-(U4A-+)
- removed copper zone on F.Cu, net ADUIO_VREF
